Commit message: Record evaluation episodes to video
eval.launch.py record_video:=true adds a 1280x720, 30 Hz (sim time) camera
looking down on the arena and a video_recorder node that reads its frames
from gz-transport, draws the episode id, elapsed time and a SOLVED/TIMEOUT
banner, and pipes them to ffmpeg (now in the image) as one mp4.

The goal marker and arena outline move from visibility bit 31 to 27: bits
28-31 are gz-rendering's own and cameras never rendered them.

File: src/limo_gz_description/urdf/limo.urdf.xacro (robot description, xacro)
@@ -8,6 +8,7 @@
   0.15 m above it, laser_link at (0.103, 0, -0.034) from base_link, i.e. 0.116 m above the floor.
   robot_index selects the robot's own visibility bit (1 << robot_index): its lidar masks that
-  bit out, so a robot never sees its own body, while the other robots' lidars still do. Bit 31
-  is reserved for overlay visuals (goal marker, arena lines) that no lidar should see.
+  bit out, so a robot never sees its own body, while the other robots' lidars still do. Bit 27
+  is reserved for overlay visuals (goal marker, arena lines) that no lidar should see; bits
+  28-31 are gz-rendering's own (cameras never render them).
   Leave <collision>/<visual> unnamed: sdformat's URDF parser matches <gazebo reference> blocks
   (friction, visibility flags) to collisions/visuals by their generated names, and silently
@@ -33,5 +34,5 @@
   <xacro:property name="max_ang_acc" value="$(arg max_angular_acceleration)"/>
   <xacro:property name="vis_flags" value="${2 ** int(robot_index)}"/>
-  <xacro:property name="lidar_mask" value="${(2 ** 31 - 1) ^ vis_flags}"/>
+  <xacro:property name="lidar_mask" value="${(2 ** 27 - 1) ^ vis_flags}"/>
   <!-- Body -->
   <xacro:property name="body_x" value="0.322"/>

File: src/pusht_gz/models/tee.sdf.xacro (robot description, xacro)
@@ -5,5 +5,5 @@
   floor), mass split between the boxes by area, inertia by the parallel-axis theorem.
   goal:=true gives the goal marker instead: static, visual only, a flat translucent T on the
-  floor, on visibility bit 31 so no lidar sees it.
+  floor, on visibility bit 27 so no lidar sees it.
 -->
 <sdf version="1.9" xmlns:xacro="http://ros.org/wiki/xacro">
@@ -89,5 +89,5 @@
         <cast_shadows>false</cast_shadows>
         <transparency>0.5</transparency>
-        <visibility_flags>2147483648</visibility_flags>
+        <visibility_flags>134217728</visibility_flags>
         <material>
           <ambient>0.1 0.8 0.2 1</ambient>

File: src/pusht_gz/worlds/pusht.sdf.xacro (robot description, xacro)
@@ -2,5 +2,5 @@
 <!--
   Push-T world: flat floor, sun, 1 ms physics. No walls (swarp's walls are invisible to the
-  lidar and only clamp positions); the arena outline is drawn on visibility bit 31, which no
+  lidar and only clamp positions); the arena outline is drawn on visibility bit 27, which no
   lidar sees. rtf:=0 runs as fast as possible.
 -->
@@ -11,4 +11,6 @@
   <xacro:arg name="arena_half" default="2.0"/>
   <xacro:arg name="floor_mu" default="1.0"/>
+  <xacro:arg name="camera" default="false"/>
+  <xacro:arg name="camera_rate" default="30"/>
   <xacro:property name="half" value="$(arg arena_half)"/>
   <world name="$(arg world_name)">
@@ -63,5 +65,5 @@
             <geometry><box><size>${lx} ${ly} 0.002</size></box></geometry>
             <cast_shadows>false</cast_shadows>
-            <visibility_flags>2147483648</visibility_flags>
+            <visibility_flags>134217728</visibility_flags>
             <material>
               <ambient>0.2 0.2 0.6 1</ambient>
@@ -76,4 +78,24 @@
       </link>
     </model>
+    <!-- Video camera (camera:=true): 1280x720 at camera_rate Hz of sim time on gz topic
+         /video/image, looking down at the arena from the -y side, 63 deg below horizontal. -->
+    <xacro:if value="$(arg camera)">
+      <model name="video_camera">
+        <static>true</static>
+        <pose>0 -3.1 5.4 0 1.1 1.5708</pose>
+        <link name="link">
+          <sensor name="video" type="camera">
+            <always_on>true</always_on>
+            <update_rate>$(arg camera_rate)</update_rate>
+            <topic>/video/image</topic>
+            <camera>
+              <horizontal_fov>1.15</horizontal_fov>
+              <image><width>1280</width><height>720</height><format>R8G8B8</format></image>
+              <clip><near>0.1</near><far>50</far></clip>
+            </camera>
+          </sensor>
+        </link>
+      </model>
+    </xacro:if>
   </world>
 </sdf>

Commit message: Add the real Limo bringup: onboard safety bridge, pose sources, AMCL in Gazebo
- limo_bridge (runs onboard on Foxy and Humble, rclpy + stdlib): robot_bridge clamps the
  policy's command to the trained limits, zeroes the chassis 0.3 s after the last command
  (20 Hz), on a latched /estop and past the arena edge, has a dry_run shadow mode, relays
  the driver's scan and odometry under /robot_i/ with prefixed frames (odom_yaw_scale
  corrects the skid steer's turn overestimate), and sends zeros on SIGINT/SIGTERM.
  robot.launch.py starts limo_base and the T-mini Pro remapped under /robot_i/limo/;
  amcl.launch.py runs a namespaced nav2 AMCL.
- policy_node publishes a zero twist on SIGINT/SIGTERM (rclpy without its own signal
  handler), republishes the held command every scan to feed the watchdog, drops returns
  below the checkpoint's lidar_min_range and blanks rays outside lidar_fov as swarp does.
- Gazebo runs the same robot_bridge between the policies and the DiffDrive; the Limo has
  the measured specs (4.8 kg, T-mini Pro: 400 samples, 0.02-12 m, sigma 0.015, lidar_fov).
- limo_real (laptop): mocap_relay, amcl_relay, fake_mocap, the operator console, pose_error,
  measurement scripts (firmware timeout, step response, static scan, lidar rate),
  poses.launch.py and laptop.launch.py; mocap_msgs copied from mocap4ros2.
- eval.launch.py pose_source:=gt|amcl|mocap; landmarks outside the arena and the map
  rasterized from them; the episode manager scores on ground truth and re-initialises
  AMCL after each teleport.
- docs/real_robot.md: networking, install, and the step-by-step checklist; results.md:
  ground truth 19/20 vs AMCL 15/20 on L5s.

File: src/limo_gz_description/urdf/limo.urdf.xacro (robot description, xacro)
@@ -3,5 +3,5 @@
   AgileX Limo (4WD skid steer) for Gazebo Harmonic.
   Every link, joint and frame is prefixed with "<robot_name>/", every topic lives under
-  "/<robot_name>/". Dimensions follow the AgileX spec: 0.322 x 0.220 x 0.251 m, 4.2 kg,
+  "/<robot_name>/". Dimensions follow the AgileX spec: 0.322 x 0.220 x 0.251 m, 4.8 kg,
   wheel radius 0.045 m, wheelbase 0.2 m, track 0.172 m.
   Frames (HO-MPC convention): base_footprint on the floor below the body centre, base_link
@@ -27,5 +27,11 @@
   <xacro:arg name="wheel_mu_lateral" default="0.2"/>
   <xacro:arg name="body_mu" default="0.1"/>
-  <xacro:arg name="lidar_noise_stddev" default="0.01"/>
+  <xacro:arg name="lidar_noise_stddev" default="0.015"/>
+  <xacro:arg name="lidar_samples" default="400"/>
+  <xacro:arg name="lidar_min_range" default="0.02"/>
+  <xacro:arg name="lidar_max_range" default="12.0"/>
+  <xacro:arg name="lidar_rate" default="10"/>
+  <xacro:arg name="lidar_fov" default="6.283185307179586"/>
+  <xacro:arg name="cmd_vel_topic" default=""/>
   <xacro:property name="name" value="$(arg robot_name)"/>
   <xacro:property name="p" value="$(arg robot_name)/"/>
@@ -41,6 +47,6 @@
   <xacro:property name="body_bottom" value="0.020"/>
   <xacro:property name="base_link_z" value="0.15"/>
-  <xacro:property name="body_mass" value="3.4"/>
-  <!-- Wheels: 4 x 0.2 kg, so the robot weighs 4.2 kg -->
+  <xacro:property name="body_mass" value="4.0"/>
+  <!-- Wheels: 4 x 0.2 kg, so the robot weighs 4.8 kg -->
   <xacro:property name="wheel_radius" value="0.045"/>
   <xacro:property name="wheel_width" value="0.045"/>
@@ -48,4 +54,15 @@
   <xacro:property name="wheelbase" value="0.2"/>
   <xacro:property name="track" value="0.172"/>
+  <!-- Lidar: EAI T-mini Pro, lidar_samples per full turn. A field of view below 2 pi (the
+       chassis blocking the rear) keeps the rays within fov / 2 of the heading. -->
+  <xacro:property name="lidar_n" value="${int($(arg lidar_samples))}"/>
+  <xacro:property name="lidar_fov" value="${float($(arg lidar_fov))}"/>
+  <xacro:property name="lidar_full" value="${lidar_fov >= 2 * pi - 1e-6}"/>
+  <xacro:property name="lidar_rays" value="${lidar_n if lidar_full else int(round(lidar_n * lidar_fov / (2 * pi))) + 1}"/>
+  <xacro:property name="lidar_min_angle" value="${-pi if lidar_full else -lidar_fov / 2}"/>
+  <xacro:property name="lidar_max_angle" value="${pi - 2 * pi / lidar_n if lidar_full else lidar_fov / 2}"/>
+  <!-- DiffDrive's command topic: the safety bridge's output (limo_bridge robot_bridge), as
+       on the real robot, where limo_base's /cmd_vel is remapped to /<robot>/limo/cmd_vel. -->
+  <xacro:property name="cmd_topic" value="${'$(arg cmd_vel_topic)' or '/' + name + '/limo/cmd_vel'}"/>
   <!-- Lidar mount, from base_link -->
   <xacro:property name="lidar_x" value="0.103"/>
@@ -183,5 +200,5 @@
       <topic>/${name}/scan</topic>
       <gz_frame_id>${p}laser_link</gz_frame_id>
-      <update_rate>10</update_rate>
+      <update_rate>$(arg lidar_rate)</update_rate>
       <always_on>true</always_on>
       <visualize>false</visualize>
@@ -189,9 +206,9 @@
         <scan>
           <horizontal>
-            <!-- 1 deg steps over the full circle, no duplicate ray at +-pi -->
-            <samples>360</samples>
+            <!-- 2 pi / lidar_samples steps; over the full circle no duplicate ray at +-pi -->
+            <samples>${lidar_rays}</samples>
             <resolution>1</resolution>
-            <min_angle>${-pi}</min_angle>
-            <max_angle>${pi - 2 * pi / 360}</max_angle>
+            <min_angle>${lidar_min_angle}</min_angle>
+            <max_angle>${lidar_max_angle}</max_angle>
           </horizontal>
           <vertical>
@@ -203,6 +220,6 @@
         </scan>
         <range>
-          <min>0.10</min>
-          <max>8.0</max>
+          <min>$(arg lidar_min_range)</min>
+          <max>$(arg lidar_max_range)</max>
           <resolution>0.01</resolution>
         </range>
@@ -241,6 +258,6 @@
       <max_angular_acceleration>${max_ang_acc}</max_angular_acceleration>
       <min_angular_acceleration>${-max_ang_acc}</min_angular_acceleration>
-      <topic>/${name}/cmd_vel</topic>
-      <odom_topic>/${name}/odom</odom_topic>
+      <topic>${cmd_topic}</topic>
+      <odom_topic>/${name}/limo/odom</odom_topic>
       <odom_publish_frequency>$(arg odom_publish_frequency)</odom_publish_frequency>
       <tf_topic>/${name}/odom_tf</tf_topic>
